File: RP2350b_Console/RP2350b_Console.kicad_sch (KiCad schematic)
At the start: 46 parts, among them J1 USB_B_Micro, J4 SM03B-SRSS-TB, J5 Conn_01x08_MountingPin, SW1 SW_Push, SW2 SW_Push, SW3 RotaryEncoder_Switch_MP, SW4 RotaryEncoder_Switch_MP, U1 RP2350_80QFN, U2 NCP1117-3.3_SOT223, U3 LY68L6400SLIT, U5 W25Q128, Y1 ABM8-272-T3

Commit message: half way through second version
Parts:
- removed C1, C19, C5: 10u, Capacitor_SMD:C_0805_2012Metric, symbol Device:C
- removed C10, C9: 4.7u, Capacitor_SMD:C_0402_1005Metric, symbol Device:C
- removed C11, C12, C13, C14, C15, C16, C17, C18, C2, C20, C21, C8: 100n, Capacitor_SMD:C_0402_1005Metric, symbol Device:C
- removed C22: DNF, Capacitor_SMD:C_0402_1005Metric, symbol Device:C
- removed C3, C4: 15p, Capacitor_SMD:C_0402_1005Metric, symbol Device:C
- removed C6, C7: 4.7u, RP2350_80QFN_minimal:C_0402_1005Metric_small_pads, symbol Device:C
- removed J1: USB_B_Micro, Connector_USB:USB_Micro-B_Amphenol_10103594-0001LF_Horizontal, symbol Connector:USB_B_Micro
- removed J4: SM03B-SRSS-TB, Connector_JST:JST_SH_SM03B-SRSS-TB_1x03-1MP_P1.00mm_Horizontal, symbol Connector_Generic_MountingPin:Conn_01x03_MountingPin
- removed R1, R13: 10k, Resistor_SMD:R_0402_1005Metric, symbol Device:R
- removed R10, R11: 0, Resistor_SMD:R_0402_1005Metric, symbol Device:R
- removed R2, R4, R6: 1k, Resistor_SMD:R_0402_1005Metric, symbol Device:R
- removed R3: 33, Resistor_SMD:R_0402_1005Metric, symbol Device:R
- removed R7, R8: 27, Resistor_SMD:R_0402_1005Metric, symbol Device:R
- removed U2: NCP1117-3.3_SOT223, Package_TO_SOT_SMD:SOT-223-3_TabPin2, symbol Regulator_Linear:NCP1117-3.3_SOT223
- removed Y1: ABM8-272-T3, Crystal:Crystal_SMD_3225-4Pin_3.2x2.5mm, symbol Device:Crystal_GND24
- added C1, C27, C7: 100uF, PCM_JLCPCB:C_1206, symbol PCM_JLCPCB-Capacitors:1206,100uF
- added C11, C15, C6, C8: 4.7uF, PCM_JLCPCB:C_0402, symbol PCM_JLCPCB-Capacitors:0402,4.7uF
- added C12, C13, C14, C2, C23, C28, C3, C30, C31, C32, C33, C34, C35, C4: 100nF, PCM_JLCPCB:C_0402, symbol PCM_JLCPCB-Capacitors:0402,100nF,(2)
- added C22, C29: 15pF, PCM_JLCPCB:C_0402, symbol PCM_JLCPCB-Capacitors:0402,15pF
- added C24: 1nF, PCM_JLCPCB:C_0402, symbol PCM_JLCPCB-Capacitors:0402,1nF
- added C25: 10pF, PCM_JLCPCB:C_0402, symbol PCM_JLCPCB-Capacitors:0402,10pF
- added C26: 22uF, PCM_JLCPCB:C_0805, symbol PCM_JLCPCB-Capacitors:0805,22uF
- added C5: 2.7nF, PCM_JLCPCB:C_0603, symbol PCM_JLCPCB-Capacitors:0603,2.7nF
- added D1: SS24F, PCM_JLCPCB:D_SMAF, symbol PCM_JLCPCB-Diodes:Schottky,SS24F
- added D2: Green, PCM_JLCPCB:D_0805, symbol PCM_JLCPCB-Diodes:LED,0805,Green
- added D3: Red, PCM_JLCPCB:D_0603, symbol PCM_JLCPCB-Diodes:LED,0603,Red
- added H1, H2, H3, H4: MountingHole, MountingHole:MountingHole_2.2mm_M2_Pad_TopBottom, symbol Mechanical:MountingHole_Pad
- added J1: Conn_01x03, Connector_PinHeader_2.54mm:PinHeader_1x03_P2.54mm_Vertical, symbol Connector_Generic:Conn_01x03
- added J2: Connector, USB-TYPE-C-16P, PCM_JLCPCB:TYPE-C-SMD_HX-TYPE-C-16PIN, symbol PCM_JLCPCB-Extended:Connector, USB-TYPE-C-16P
- added L2: 2.7uH, Inductor_SMD:Bourns SRP7028AA-2R7M, symbol Device:L
- added R1, R11, R15: 10kΩ, PCM_JLCPCB:R_0402, symbol PCM_JLCPCB-Resistors:0402,10kΩ
- added R10, R17: 0Ω, PCM_JLCPCB:R_0402, symbol PCM_JLCPCB-Resistors:0402,0Ω
- added R12, R5: 5.1kΩ, PCM_JLCPCB:R_0402, symbol PCM_JLCPCB-Resistors:0402,5.1kΩ
- added R13, R2, R4: 1kΩ, PCM_JLCPCB:R_0402, symbol PCM_JLCPCB-Resistors:0402,1kΩ
- added R14: 24kΩ, PCM_JLCPCB:R_0402, symbol PCM_JLCPCB-Resistors:0402,24kΩ
- added R16: 3.3kΩ, PCM_JLCPCB:R_0402, symbol PCM_JLCPCB-Resistors:0402,3.3kΩ
- added R18, R8: 100Ω, PCM_JLCPCB:R_0402, symbol PCM_JLCPCB-Resistors:0402,100Ω
- added R3, R7: 27Ω, PCM_JLCPCB:R_0603, symbol PCM_JLCPCB-Resistors:0603,27Ω
- added R6: 33Ω, PCM_JLCPCB:R_0402, symbol PCM_JLCPCB-Resistors:0402,33Ω
- added U2: TPS54331DR, PCM_JLCPCB:SOIC-8_L5.0-W4.0-P1.27-LS6.0-BL, symbol PCM_JLCPCB-Power:DC-DC, Buck, 3.5-28VIN, 3A, 0.8+VOUT
- added X1: X322512MSB4SI, PCM_JLCPCB:CRYSTAL-SMD_4P-L3.2-W2.5-BL, symbol PCM_JLCPCB-Crystals:Crystal, 12MHz, 20pF
Connections:
- net +1V1: now also C11.1, C13.1, C14.1, C8.1
- net +3V3: now also C1.1, C12.1, C15.1, C2.1, C27.1, C28.1, C3.1, C30.1, C31.1, C32.1, C33.1, C34.1, C35.1, C4.1, C7.1, L2.2, R1.1, R11.1, R15.1, R6.1, R8.2
- net FLASH2_SS: now also R10.2, R11.2
- net FLASH_SS: now also R1.2, R17.2
- net GND: now also J5.MP (MountPin), C1.2, C11.2, C12.2, C13.2, C14.2, C15.2, C2.2, C22.2, C24.2, C25.2, C26.2, C27.2, C28.2, C29.2, C3.2, C30.2, C31.2, C32.2, C33.2, C34.2, C35.2, C4.2, C5.2, C6.2, C7.2, C8.2, D1.2, D2.1, D3.1, H1.1, H2.1, H3.1, H4.1, J1.3 (Pin_3), J2.A12B1 (GND), J2.B12A1 (GND), J2.S1 (SHIELD), R12.2, R16.2, R2.1, R5.2, U2.7 (GND), X1.2 (GND), X1.4 (GND)
- net GPIO0: now also R10.1
- net GPIO1: now also R18.2
- net QSPI_SS: now also R17.1, R4.2
- net SWCLK: now also J1.1 (Pin_1)
- net SWD: now also J1.2 (Pin_2)
- net USB_D+: now also J2.A6 (D+), J2.B6 (D+), R7.2
- net USB_D-: now also J2.A7 (D-), J2.B7 (D-), R3.2
- net VBUS: now also C26.1, J2.A9B4 (VBUS), J2.B9A4 (VBUS), U2.2 (VIN)
- net VREG_AVDD: now also C6.1, R6.2
- net XIN: now also C29.1, X1.1 (OSC)
- net XOUT: now also R13.2
- net ~{USB_BOOT}: now also R4.1
- net at U1.67 (USB_DP): now also R7.1
- net at U1.66 (USB_DM): now also R3.1
- net at SW2.1: now also R2.2
- new net: J2.B5 (CC2), R12.1
- new net: D2.2, R8.1
- new net: C23.1, D1.1, L2.1, U2.8 (PH)
- new net: C23.2, U2.1 (BOOT)
- new net: R15.2, R16.1, U2.5 (VSENSE)
- new net: C25.1, R14.1, U2.6 (COMP)
- new net: C24.1, R14.2
- new net: J2.A5 (CC1), R5.1
- new net: C5.1, U2.4 (SS)
- new net: C22.1, R13.1, X1.3 (OSC)
- new net: D3.2, R18.1
- no-connect marks 1 -> 3
Other:
- note added: "Decoupling Caps"
- note added: "LEDS"
- note added: "USB C"
- moved on the sheet: J5, L1, R9, SW1, SW2, SW3, SW4, U1, U3, U5
