File: RP2350b_Console/RP2350b_Console.kicad_sch (KiCad schematic)
At the start: 63 parts, among them J2 Connector, USB-TYPE-C-16P, J5 Conn_01x08_MountingPin, SW1 SW_Push, SW2 SW_Push, SW3 RotaryEncoder_Switch_MP, SW4 RotaryEncoder_Switch_MP, U1 RP2350_80QFN, U2 TPS54331DR, U3 LY68L6400SLIT, U5 W25Q128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

Commit message: updates - build 1
Parts:
- removed L1: 3.3u, RP2350_80QFN_minimal:L_pol_2016, symbol Device:L
- added L1: 3.3uH, Inductor_SMD:IND-SMD_L2.0-W1.6_AOTA-B201610S3R3-101-T, symbol Custom:AOTA-B201610S3R3-101-T
Connections:
- net +1V1: now also L1.2
- net QSPI2_SS: now also U1.77 (GPIO0); no longer U1.6 (GPIO8)
- net USER_LED: now also U1.6 (GPIO8); no longer U1.77 (GPIO0)
- net VREG_LX: now also L1.1
Other:
- title: RP2350B QFN80 Board w/ Screen and Rotary Encoders -> RP2350b Console
Changed lines of the file:
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@@
 	(paper "A3")
 	(title_block
-		(title "RP2350B QFN80 Board w/ Screen and Rotary Encoders")
-		(date "2025-08-23")
+		(title "RP2350b Console")
+		(date "2025-09-28")
 		(rev "REV1")
 		(company "Kirill Kobyakov")
 	)
 	(circle
-		(center 146.685 137.16)
+		(center 149.225 135.255)
 		(radius 0.635)
 		(stroke
@@
 	)
 	(junction
+		(at 132.715 133.35)
+		(diameter 0)
+		(color 0 0 0 0)
+	)
+	(junction
 		(at 62.865 131.445)
 		(diameter 0)
@@
 	)
 	(junction
-		(at 147.955 133.985)
+		(at 147.955 133.35)
 		(diameter 0)
 		(color 0 0 0 0)
@@
 	)
 	(junction
-		(at 132.715 133.985)
-		(diameter 0)
-		(color 0 0 0 0)
-	)
-	(junction
 		(at 215.265 112.395)
 		(diameter 0)
@@
 	(wire
 		(pts
-			(xy 155.575 133.985) (xy 147.955 133.985)
+			(xy 155.575 133.35) (xy 147.955 133.35)
 		)
 		(stroke
@@
 	(wire
 		(pts
-			(xy 132.715 132.715) (xy 132.715 133.985)
+			(xy 132.715 132.715) (xy 132.715 133.35)
 		)
 		(stroke
@@
 	(wire
 		(pts
-			(xy 147.955 144.145) (xy 147.955 142.875)
+			(xy 59.69 202.565) (xy 63.5 202.565)
 		)
 		(stroke
@@
 	(wire
 		(pts
-			(xy 59.69 202.565) (xy 63.5 202.565)
+			(xy 147.955 133.35) (xy 147.955 133.985)
 		)
 		(stroke
@@
 	(wire
 		(pts
-			(xy 155.575 141.605) (xy 155.575 133.985)
+			(xy 155.575 141.605) (xy 155.575 133.35)
 		)
 		(stroke
@@
 	(wire
 		(pts
+			(xy 132.715 133.35) (xy 132.715 135.255)
+		)
+		(stroke
+			(width 0)
+			(type default)
+		)
+	)
+	(wire
+		(pts
 			(xy 271.145 99.695) (xy 271.145 102.235)
 		)
@@
 	(wire
 		(pts
-			(xy 132.715 133.985) (xy 147.955 133.985)
+			(xy 132.715 133.35) (xy 147.955 133.35)
 		)
 		(stroke
@@
 	(wire
 		(pts
-			(xy 147.955 133.985) (xy 147.955 135.255)
-		)
-		(stroke
-			(width 0)
-			(type default)
-		)
-	)
-	(wire
-		(pts
 			(xy 207.645 112.395) (xy 210.185 112.395)
 		)
@@
 	(wire
 		(pts
-			(xy 132.715 135.255) (xy 132.715 133.985)
-		)
-		(stroke
-			(width 0)
-			(type default)
-		)
-	)
-	(wire
-		(pts
 			(xy 172.72 46.99) (xy 149.225 46.99)
 		)
@@
 		)
 	)
+	(label "USER_LED"
+		(at 263.525 163.195 180)
+		(effects
+			(font
+				(size 1.27 1.27)
+			)
+			(justify right bottom)
+		)
+	)
+	(label "QSPI2_SS"
+		(at 263.525 142.875 180)
+		(effects
+			(font
+				(size 1.27 1.27)
+			)
+			(justify right bottom)
+		)
+	)
 	(label "Screen_DIN"
 		(at 287.6395 56.515 0)
@@
 		)
 	)
-	(label "QSPI2_SS"
-		(at 263.525 163.195 180)
-		(effects
-			(font
-				(size 1.27 1.27)
-			)
-			(justify right bottom)
-		)
-	)
 	(label "QSPI_SD2"
 		(at 50.8 136.525 0)
@@
 		)
 	)
-	(label "USER_LED"
-		(at 263.525 142.875 180)
-		(effects
-			(font
-				(size 1.27 1.27)
-			)
-			(justify right bottom)
-		)
-	)
 	(label "Screen_BL"
 		(at 287.6395 43.815 0)
@@
 	)
 	(symbol
-		(lib_id "Device:L")
-		(at 147.955 139.065 0)
-		(unit 1)
-		(exclude_from_sim no)
-		(in_bom yes)
-		(on_board yes)
-		(dnp no)
-		(fields_autoplaced yes)
-		(property "Reference" "L1"
-			(at 149.225 137.795 0)
-			(effects
-				(font
-					(size 1.27 1.27)
-				)
-				(justify left)
-			)
-		)
-		(property "Value" "3.3u"
-			(at 149.225 140.335 0)
-			(effects
-				(font
-					(size 1.27 1.27)
-				)
-				(justify left)
-			)
-		)
-		(property "Footprint" "RP2350_80QFN_minimal:L_pol_2016"
-			(at 147.955 139.065 0)
-			(effects
-				(font
-					(size 1.27 1.27)
-				)
-				(hide yes)
-			)
-		)
-		(property "Datasheet" "~"
-			(at 147.955 139.065 0)
-			(effects
-				(font
-					(size 1.27 1.27)
-				)
-				(hide yes)
-			)
-		)
-		(property "Description" ""
-			(at 147.955 139.065 0)
-			(effects
-				(font
-					(size 1.27 1.27)
-				)
-			)
-		)
-		(pin "1"
-		)
-		(pin "2"
-		)
-		(instances
-			(project "RP2350_80QFN_minimal"
-				(path "/94683f5c-9cd9-448e-be96-9792537b5cb8"
-					(reference "L1")
-					(unit 1)
-				)
-			)
-		)
-	)
-	(symbol
 		(lib_id "PCM_JLCPCB-Capacitors:0402,100nF,(2)")
 		(at 237.49 106.045 0)
@@
 					(unit 1)
 				)
+			)
+		)
+	)
+	(symbol
+		(lib_id "Custom:AOTA-B201610S3R3-101-T")
+		(at 147.955 139.065 90)
+		(unit 1)
+		(exclude_from_sim no)
+		(in_bom yes)
+		(on_board yes)
+		(dnp no)
+		(fields_autoplaced yes)
+		(property "Reference" "L1"
+			(at 148.59 137.7949 90)
+			(effects
+				(font
+					(size 1.27 1.27)
+				)
+				(justify right)
+			)
+		)
+		(property "Value" "3.3uH"
+			(at 148.59 140.3349 90)
+			(effects
+				(font
+					(size 1.27 1.27)
+				)
+				(justify right)
+			)
+		)
+		(property "Footprint" "Inductor_SMD:IND-SMD_L2.0-W1.6_AOTA-B201610S3R3-101-T"
+			(at 147.955 139.065 0)
+			(effects
+				(font
+					(size 1.27 1.27)
+				)
+				(hide yes)
+			)
+		)
+		(property "Datasheet" "https://item.szlcsc.com/datasheet/AOTA-B201610S3R3-101-T/44392932.html"
+			(at 147.955 139.065 0)
+			(effects
+				(font
+					(size 1.27 1.27)
+				)
+				(hide yes)
+			)
+		)
+		(property "Description" ""
+			(at 147.955 139.065 0)
+			(effects
+				(font
+					(size 1.27 1.27)
+				)
+				(hide yes)
+			)
+		)
+		(property "Manufacturer Part" "AOTA-B201610S3R3-101-T"
+			(at 147.955 139.065 0)
+			(effects
+				(font
+					(size 1.27 1.27)
+				)
+				(hide yes)
+			)
+		)
+		(property "Manufacturer" "ABRACON"
+			(at 147.955 139.065 0)
+			(effects
+				(font
+					(size 1.27 1.27)
+				)
+				(hide yes)
+			)
+		)
+		(property "Supplier Part" "C42411119"
+			(at 147.955 139.065 0)
+			(effects
+				(font
+					(size 1.27 1.27)
+				)
+				(hide yes)
+			)
+		)
+		(property "Supplier" "LCSC"
+			(at 147.955 139.065 0)
+			(effects
+				(font
+					(size 1.27 1.27)
+				)
+				(hide yes)
+			)
+		)
+		(property "LCSC Part Name" "AOTA-B201610S3R3-101-T"
+			(at 147.955 139.065 0)
+			(effects
+				(font
+					(size 1.27 1.27)
+				)
+				(hide yes)
+			)
+		)
+		(pin "2"
+		)
+		(pin "1"
+		)
+		(instances
+			(project ""
+				(path "/94683f5c-9cd9-448e-be96-9792537b5cb8"
+					(reference "L1")
+					(unit 1)
+				)
