File: RP2350b_Console/RP2350b_Console.kicad_pcb (KiCad board)
At the start: 2 copper layers, 100 x 45 mm, 46 parts, among them J1 USB_B_Micro, J4 SM03B-SRSS-TB, J5 Conn_01x08_MountingPin, SW1 SW_Push, SW2 SW_Push, SW3 RotaryEncoder_Switch_MP, SW4 RotaryEncoder_Switch_MP, U1 RP2350_80QFN, U2 NCP1117-3.3_SOT223, U3 LY68L6400SLIT, U5 W25Q128, Y1 ABM8-272-T3

Commit message: half way through second version
Parts:
- removed C10, C9: 4.7u, Capacitor_SMD:C_0402_1005Metric
- removed C16, C17, C18, C20, C21: 100n, Capacitor_SMD:C_0402_1005Metric
- removed C19: 10u, Capacitor_SMD:C_0805_2012Metric
- removed J4: SM03B-SRSS-TB, Connector_JST:JST_SH_SM03B-SRSS-TB_1x03-1MP_P1.00mm_Horizontal
- removed Y1: ABM8-272-T3, Crystal:Crystal_SMD_3225-4Pin_3.2x2.5mm
- added C23: 100nF, PCM_JLCPCB:C_0402, F.Cu at (103.6, 117.2)
- added C24: 1nF, PCM_JLCPCB:C_0402, F.Cu at (110.0, 120.1)
- added C25: 10pF, PCM_JLCPCB:C_0402, F.Cu at (108.2, 120.6)
- added C26: 22uF, PCM_JLCPCB:C_0805, F.Cu at (98.5, 118.8)
- added C27: 100uF, PCM_JLCPCB:C_1206, F.Cu at (122.0, 122.9)
- added C28: 100nF, PCM_JLCPCB:C_0402, F.Cu at (156.6, 125.1)
- added C29: 15pF, PCM_JLCPCB:C_0402, F.Cu at (88.9, 140.6)
- added C30: 100nF, PCM_JLCPCB:C_0402, F.Cu at (159.5, 114.0)
- added C31: 100nF, PCM_JLCPCB:C_0402, F.Cu at (159.5, 115.9)
- added C32: 100nF, PCM_JLCPCB:C_0402, F.Cu at (159.5, 117.7)
- added C33: 100nF, PCM_JLCPCB:C_0402, F.Cu at (159.5, 119.6)
- added C34: 100nF, PCM_JLCPCB:C_0402, F.Cu at (159.5, 121.4)
- added C35: 100nF, PCM_JLCPCB:C_0402, F.Cu at (159.5, 123.3)
- added D1: SS24F, PCM_JLCPCB:D_SMAF, F.Cu at (111.4, 116.4)
- added D2: Green, PCM_JLCPCB:D_0805, F.Cu at (140.1, 141.4)
- added D3: Red, PCM_JLCPCB:D_0603, F.Cu at (166.6, 138.7)
- added H1: MountingHole, MountingHole:MountingHole_2.2mm_M2_Pad_TopBottom, F.Cu at (127.0, 113.0)
- added H2: MountingHole, MountingHole:MountingHole_2.2mm_M2_Pad_TopBottom, F.Cu at (53.0, 113.0)
- added H3: MountingHole, MountingHole:MountingHole_2.2mm_M2_Pad_TopBottom, F.Cu at (53.0, 147.0)
- added H4: MountingHole, MountingHole:MountingHole_2.2mm_M2_Pad_TopBottom, F.Cu at (127.0, 147.0)
- added J2: Connector, USB-TYPE-C-16P, PCM_JLCPCB:TYPE-C-SMD_HX-TYPE-C-16PIN, F.Cu at (90.0, 115.0)
- added L2: 2.7uH, Inductor_SMD:Bourns SRP7028AA-2R7M, F.Cu at (116.6, 121.0)
- added R12: 5.1kΩ, PCM_JLCPCB:R_0402, F.Cu at (88.3, 119.8)
- added R14: 24kΩ, PCM_JLCPCB:R_0402, F.Cu at (110.0, 121.1)
- added R15: 10kΩ, PCM_JLCPCB:R_0402, F.Cu at (111.9, 123.9)
- added R16: 3.3kΩ, PCM_JLCPCB:R_0402, F.Cu at (111.9, 121.9)
- added R17: 0Ω, PCM_JLCPCB:R_0402, F.Cu at (61.1, 129.2)
- added R18: 100Ω, PCM_JLCPCB:R_0402, F.Cu at (163.7, 139.0)
- added R5: 5.1kΩ, PCM_JLCPCB:R_0402, F.Cu at (91.3, 119.8)
- added X1: X322512MSB4SI, PCM_JLCPCB:CRYSTAL-SMD_4P-L3.2-W2.5-BL, F.Cu at (90.0, 143.1)
- C1: value 10u -> 100uF; footprint Capacitor_SMD:C_0805_2012Metric -> PCM_JLCPCB:C_1206
- C11, C15, C8: value 100n -> 4.7uF; footprint Capacitor_SMD:C_0402_1005Metric -> PCM_JLCPCB:C_0402
- C12, C13, C14, C2: value 100n -> 100nF; footprint Capacitor_SMD:C_0402_1005Metric -> PCM_JLCPCB:C_0402
- C22: value DNF -> 15pF; footprint Capacitor_SMD:C_0402_1005Metric -> PCM_JLCPCB:C_0402; moved to F.Cu
- C3, C4: value 15p -> 100nF; footprint Capacitor_SMD:C_0402_1005Metric -> PCM_JLCPCB:C_0402
- C5: value 10u -> 2.7nF; footprint Capacitor_SMD:C_0805_2012Metric -> PCM_JLCPCB:C_0603
- C6: value 4.7u -> 4.7uF; footprint RP2350_80QFN_minimal:C_0402_1005Metric_small_pads -> PCM_JLCPCB:C_0402
- C7: value 4.7u -> 100uF; footprint RP2350_80QFN_minimal:C_0402_1005Metric_small_pads -> PCM_JLCPCB:C_1206
- J1: value USB_B_Micro -> Conn_01x03; footprint Connector_USB:USB_Micro-B_Amphenol_10103594-0001LF_Horizontal -> Connector_PinHeader_2.54mm:PinHeader_1x03_P2.54mm_Vertical
- R1: value 10k -> 10kΩ; footprint Resistor_SMD:R_0402_1005Metric -> PCM_JLCPCB:R_0402
- R10: value 0 -> 0Ω; footprint Resistor_SMD:R_0402_1005Metric -> PCM_JLCPCB:R_0402
- R11: value 0 -> 10kΩ; footprint Resistor_SMD:R_0402_1005Metric -> PCM_JLCPCB:R_0402
- R13: value 10k -> 1kΩ; footprint Resistor_SMD:R_0402_1005Metric -> PCM_JLCPCB:R_0402
- R2, R4: value 1k -> 1kΩ; footprint Resistor_SMD:R_0402_1005Metric -> PCM_JLCPCB:R_0402
- R3: value 33 -> 27Ω; footprint Resistor_SMD:R_0402_1005Metric -> PCM_JLCPCB:R_0603
- R6: value 1k -> 33Ω; footprint Resistor_SMD:R_0402_1005Metric -> PCM_JLCPCB:R_0402
- R7: value 27 -> 27Ω; footprint Resistor_SMD:R_0402_1005Metric -> PCM_JLCPCB:R_0603
- R8: value 27 -> 100Ω; footprint Resistor_SMD:R_0402_1005Metric -> PCM_JLCPCB:R_0402
- SW1, SW2, SW3, SW4: moved to B.Cu
- U2: value NCP1117-3.3_SOT223 -> TPS54331DR; footprint Package_TO_SOT_SMD:SOT-223-3_TabPin2 -> PCM_JLCPCB:SOIC-8_L5.0-W4.0-P1.27-LS6.0-BL
- U5: moved to F.Cu
- moved R1 95.7 mm to (55.3, 122.2), turned to 0 degrees
- moved SW1 95.7 mm to (94.2, 163.1)
- moved SW2 92.0 mm to (104.8, 159.4)
- moved U5 84.8 mm to (61.5, 122.2), turned to 0 degrees
- moved R4 83.6 mm to (89.7, 162.4), turned to 0 degrees
- moved R11 80.0 mm to (66.9, 113.2)
- moved R10 78.6 mm to (69.5, 116.2)
- moved R13 77.8 mm to (90.2, 138.6), turned to 90 degrees
- moved U3 75.1 mm to (71.8, 121.2), turned to 0 degrees
- moved C22 74.6 mm to (91.1, 140.6), turned to 0 degrees
- moved R9 74.5 mm to (171.3, 149.1), turned to 0 degrees
- moved R2 65.6 mm to (105.2, 159.4), turned to 0 degrees
- moved R6 62.5 mm to (95.5, 123.4), turned to -90 degrees
- moved C12 59.8 mm to (88.8, 138.6), turned to -90 degrees
- moved C8 59.5 mm to (91.1, 138.6), turned to -90 degrees
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Connections:
- C1 pad 1: VBUS -> +3V3
- C13 pad 1: +3V3 -> +1V1
- C14 pad 1: +3V3 -> +1V1
- C22 pad 1: +3V3 -> Net-(C22-Pad1)
- C3 pad 1: /XIN -> +3V3
- C4 pad 1: Net-(C4-Pad1) -> +3V3
- C5 pad 1: +3V3 -> Net-(U2-SS)
- C6 pad 1: +3V3 -> /VREG_AVDD
- C7 pad 1: +1V1 -> +3V3
- J1 pad 1: VBUS -> /SWCLK
- J1 pad 2: /USB_D- -> /SWD
- J1 pad 3: /USB_D+ -> GND
- J5 pad MP: unconnected-(J5-MountPin-PadMP) -> GND
- R10 pad 1: /QSPI_SS -> /GPIO0
- R10 pad 2: /FLASH_SS -> /FLASH2_SS
- R11 pad 1: /GPIO0 -> +3V3
- R13 pad 1: +3V3 -> Net-(C22-Pad1)
- R13 pad 2: /FLASH2_SS -> /XOUT
- R2 pad 1: /XOUT -> GND
- R2 pad 2: Net-(C4-Pad1) -> Net-(R2-Pad2)
- R3 pad 1: +3V3 -> Net-(U1-USB_DM)
- R3 pad 2: /VREG_AVDD -> /USB_D-
- R4 pad 1: Net-(R4-Pad1) -> /~{USB_BOOT}
- R4 pad 2: GND -> /QSPI_SS
- R6 pad 1: /QSPI_SS -> +3V3
- R6 pad 2: /~{USB_BOOT} -> /VREG_AVDD
- R7 pad 1: /USB_D+ -> Net-(U1-USB_DP)
- R7 pad 2: Net-(U1-USB_DP) -> /USB_D+
- R8 pad 1: /USB_D- -> Net-(D2-Pad2)
- R8 pad 2: Net-(U1-USB_DM) -> +3V3
- SW2 pad 1: Net-(R4-Pad1) -> Net-(R2-Pad2)
- U2 pad 1: GND -> Net-(U2-BOOT)
- U2 pad 2: +3V3 -> VBUS
- U2 pad 3: VBUS -> unconnected-(U2-EN-Pad3)
Routing:
- net /RUN: track 69.0 -> 0.00 mm, vias 2 -> 0
- net /SW4_BUT: track 66.0 -> 0.00 mm
- net /SWCLK: track 61.0 -> 0.00 mm
- net /SWD: track 60.3 -> 0.00 mm
- net /SW4_P1: track 53.2 -> 0.00 mm
- net /SW4_P2: track 49.3 -> 0.00 mm
- net +3V3: track 49.5 -> 6.46 mm, vias 4 -> 0
- net GND: track 44.2 -> 12.4 mm, vias 26 -> 12
- net /SW3_BUT: track 30.8 -> 0.00 mm
- net /Screen_DIN: track 27.8 -> 0.00 mm, vias 1 -> 0
- net /QSPI_SD1: track 27.6 -> 0.00 mm, vias 1 -> 0
- net /Screen_CLK: track 26.2 -> 0.00 mm, vias 1 -> 0
- net /Screen_CS: track 26.1 -> 0.00 mm, vias 1 -> 0
- net +1V1: track 29.0 -> 3.34 mm, vias 8 -> 2
- net /Screen_DC: track 25.4 -> 0.00 mm, vias 1 -> 0
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- removed copper zone on B.Cu, net GND
Other:
- board size 100 x 45 mm -> 80 x 40 mm

Commit message: updates to project
Parts:
- removed C7: 100uF, PCM_JLCPCB:C_1206
- removed J1: Conn_01x03, Connector_PinHeader_2.54mm:PinHeader_1x03_P2.54mm_Vertical
- removed R9: DNF, Resistor_SMD:R_0402_1005Metric
- L2: footprint Inductor_SMD:Bourns SRP7028AA-2R7M -> Inductor_SMD:IND-SMD_L5.0-W5.0_FNR50XXS
- SW1, SW2: footprint Button_Switch_SMD:SW_Push_1P1T_NO_Vertical_Wuerth_434133025816 -> Button_Switch_THT:SW_1825910-6-4
- X1: value X322512MSB4SI -> ABM8-272-T3
- moved D3 105.0 mm to (64.7, 113.5), turned to -90 degrees
- moved R18 101.4 mm to (64.7, 116.7), turned to -90 degrees
- moved C28 89.4 mm to (67.2, 126.6)
- moved C30 81.5 mm to (80.5, 134.0), turned to 180 degrees
- moved C2 81.1 mm to (73.8, 127.6), turned to 180 degrees
- moved C31 78.9 mm to (84.5, 140.5), turned to -90 degrees
- moved R8 78.5 mm to (69.0, 116.6), turned to -90 degrees
- moved C14 78.2 mm to (80.5, 131.8), turned to 180 degrees
- moved D2 76.3 mm to (69.0, 113.6), turned to -90 degrees
- moved C35 75.6 mm to (83.9, 126.0), turned to -90 degrees
- moved C3 74.6 mm to (80.5, 129.5), turned to 180 degrees
- moved C4 65.7 mm to (88.3, 122.5), turned to 90 degrees
- moved C32 65.2 mm to (97.4, 137.7)
- moved C33 61.5 mm to (98.4, 127.2)
- moved C34 61.3 mm to (99.1, 132.2)
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Connections:
- R10 pad 1: /GPIO0 -> /QSPI2_SS
- R18 pad 2: /GPIO1 -> /USER_LED
- SW1 pad 2: /~{USB_BOOT} -> GND
- SW2 pad 2: /RUN -> Net-(R2-Pad2)
- SW3 pad A: /SW3_P1 -> /LQ_P1
- SW3 pad B: /SW3_P2 -> /LQ_P2
- SW3 pad S1: /SW3_BUT -> /LQ_BUT
- SW4 pad A: /SW4_P1 -> /RQ_P1
- SW4 pad B: /SW4_P2 -> /RQ_P2
- SW4 pad S1: /SW4_BUT -> /RQ_BUT
- U1 pad 21: /GPIO21 -> /RQ_BUT
- U1 pad 22: /GPIO22 -> /RQ_P1
- U1 pad 23: /GPIO23 -> /RQ_P2
- U1 pad 25: /GPIO24 -> /Screen_BL
- U1 pad 26: /GPIO25 -> /Screen_RST
- U1 pad 27: /GPIO26 -> /Screen_DC
- U1 pad 37: /GPIO29 -> /Screen_CS
- U1 pad 38: /SW4_BUT -> /Screen_CLK
- U1 pad 39: /SW4_P2 -> /Screen_DIN
- U1 pad 40: /SW4_P1 -> /GPIO32
- U1 pad 42: /GPIO33 -> /LQ_P1
- U1 pad 43: /Screen_CLK -> /LQ_P2
- U1 pad 44: /Screen_DIN -> /LQ_BUT
- U1 pad 45: /Screen_DC -> /GPIO36
- U1 pad 46: /Screen_CS -> /GPIO37
- U1 pad 47: /Screen_RST -> /GPIO38
- U1 pad 48: /Screen_BL -> /GPIO39
- U1 pad 56: /SW3_P2 -> /GPIO45_ADC5
- U1 pad 57: /SW3_P1 -> /GPIO46_ADC6
- U1 pad 58: /SW3_BUT -> /GPIO47_ADC7
- U1 pad 6: /GPIO8 -> /QSPI2_SS
- U1 pad 77: /GPIO0 -> /USER_LED
Routing:
- net +3V3: track 6.46 -> 113.7 mm, vias 0 -> 1
- net /RUN: track 0.00 -> 39.5 mm, vias 0 -> 2
- net +1V1: track 3.34 -> 36.4 mm, vias 2 -> 9
- net /USER_LED: track 0.00 -> 32.1 mm, vias 0 -> 2
- net /LQ_BUT: track 0.00 -> 31.5 mm
- net GND: track 12.4 -> 43.9 mm, vias 12 -> 40
- net /~{USB_BOOT}: track 0.00 -> 30.5 mm, vias 0 -> 2
- net /RQ_BUT: track 0.00 -> 29.6 mm
- net /QSPI_SD3: track 0.00 -> 26.3 mm, vias 0 -> 3
- net /QSPI_SCLK: track 0.00 -> 25.7 mm, vias 0 -> 3
- net /QSPI_SD0: track 0.00 -> 25.0 mm, vias 0 -> 3
- net /QSPI_SD2: track 0.00 -> 24.2 mm, vias 0 -> 3
- net /QSPI_SD1: track 0.00 -> 23.6 mm, vias 0 -> 3
- net /RQ_P2: track 0.00 -> 18.2 mm
- net /LQ_P1: track 0.00 -> 16.7 mm
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- added copper zone on B.Cu, net GND

Commit message: updates - build 1
Parts:
- L1: value 3.3u -> 3.3uH; footprint RP2350_80QFN_minimal:L_pol_2016 -> Inductor_SMD:IND-SMD_L2.0-W1.6_AOTA-B201610S3R3-101-T
- moved R17 4.44 mm to (79.4, 127.9)
- moved C35 1.05 mm to (84.8, 125.5), turned to 180 degrees
- moved R4 1.02 mm to (82.1, 128.1)
- moved L1 0.17 mm to (93.1, 123.5), turned to 180 degrees
Connections:
- L1 pad 1: +1V1 -> /VREG_LX
- L1 pad 2: /VREG_LX -> +1V1
- U1 pad 6: /QSPI2_SS -> /USER_LED
- U1 pad 77: /USER_LED -> /QSPI2_SS
Routing:
- net +3V3: track 113.7 -> 107.1 mm
- net /FLASH_SS: track 9.44 -> 4.62 mm
- net /QSPI_SS: track 8.83 -> 11.6 mm
- net /QSPI2_SS: track 16.1 -> 18.6 mm
- net /QSPI_SD3: track 26.3 -> 28.4 mm, vias 3 -> 0
- net GND: track 43.9 -> 46.0 mm, vias 40 -> 38
- net /QSPI_SD0: track 25.0 -> 23.4 mm, vias 3 -> 0
- net /QSPI_SD1: track 23.6 -> 25.2 mm, vias 3 -> 0
- net /QSPI_SD2: track 24.2 -> 22.9 mm, vias 3 -> 0
- net /QSPI_SCLK: track 25.7 -> 26.5 mm, vias 3 -> 0
- net /USER_LED: track 32.1 -> 31.6 mm
- net /~{USB_BOOT}: track 30.5 -> 30.9 mm, vias 2 -> 0
- net +1V1: vias 9 -> 10
Other:
- board text added: "PWR LED"
- board text added: "USER LED"
