File: Hardware/RP2350b_Console/RP2350b_Console.kicad_pcb (KiCad board)
At the start: 2 copper layers, 80 x 40 mm, 63 parts, among them J2 Connector, USB-TYPE-C-16P, J5 Conn_01x08_MountingPin, SW1 SW_Push, SW2 SW_Push, SW3 RotaryEncoder_Switch_MP, SW4 RotaryEncoder_Switch_MP, U1 RP2350_80QFN, U2 TPS54331DR, U3 LY68L6400SLIT, U5 W25Q128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

Commit message: updates
Parts:
- removed C23: 100nF, PCM_JLCPCB:C_0402
- removed C24: 1nF, PCM_JLCPCB:C_0402
- removed C25: 10pF, PCM_JLCPCB:C_0402
- removed C26: 22uF, PCM_JLCPCB:C_0805
- removed C27: 100uF, PCM_JLCPCB:C_1206
- removed D1: SS24F, PCM_JLCPCB:D_SMAF
- added C10: 22uF, PCM_JLCPCB:C_0603, F.Cu at (114.2, 123.8)
- added C16: 22uF, PCM_JLCPCB:C_0603, F.Cu at (114.2, 125.1)
- added C17: 22uF, PCM_JLCPCB:C_0603, F.Cu at (98.3, 118.5)
- added C18: 1uF, PCM_JLCPCB:C_0402, F.Cu at (98.0, 117.4)
- added C19: 100nF, PCM_JLCPCB:C_0402, F.Cu at (105.0, 136.1)
- added C7: 100nF, PCM_JLCPCB:C_0402, F.Cu at (110.1, 120.8)
- added C9: 10uF, PCM_JLCPCB:C_0603, F.Cu at (114.2, 122.5)
- added D5: Red, PCM_JLCPCB:D_0603, F.Cu at (103.0, 122.4)
- added R19: 47kΩ, PCM_JLCPCB:R_0603, F.Cu at (106.9, 119.4)
- added R20: 1.5kΩ, PCM_JLCPCB:R_0603, F.Cu at (108.2, 119.4)
- added R21: 100kΩ, PCM_JLCPCB:R_0603, F.Cu at (104.4, 134.4)
- added R22: 100kΩ, PCM_JLCPCB:R_0603, F.Cu at (107.5, 135.8)
- added R9: 1MΩ, PCM_JLCPCB:R_0603, F.Cu at (110.5, 123.8)
- added SW6: ~, RP2350_Console_Parts_lib:SW-TH_MK-12D18-G040, F.Cu at (112.5, 113.5)
- added U4: ~, RP2350_Console_Parts_lib:MSOP-10_L3.0-W3.0-P0.50-LS5.0-BL-EP, F.Cu at (103.0, 119.7)
- C1: value 100uF -> 22uF; footprint PCM_JLCPCB:C_1206 -> PCM_JLCPCB:C_0603
- C5: value 2.7nF -> 10uF
- J5: footprint Display:Seeed 1.69 Inch LCD Module -> RP2350_Console_Parts_lib:Seeed 1.69 Inch LCD Module; moved to F.Cu
- L1: footprint Inductor_SMD:IND-SMD_L2.0-W1.6_AOTA-B201610S3R3-101-T -> RP2350_Console_Parts_lib:IND-SMD_L2.0-W1.6_AOTA-B201610S3R3-101-T
- L2: value 2.7uH -> 1.5uH; footprint Inductor_SMD:IND-SMD_L5.0-W5.0_FNR50XXS -> RP2350_Console_Parts_lib:IND-SMD_L4.0-W4.0-A
- R14: value 24kΩ -> 1MΩ; footprint PCM_JLCPCB:R_0402 -> PCM_JLCPCB:R_0603
- R15: value 10kΩ -> 1kΩ
- R16: value 3.3kΩ -> 2kΩ
- SW1, SW2: footprint Button_Switch_THT:SW_1825910-6-4 -> RP2350_Console_Parts_lib:SW-TH_4P-L6.0-W6.0-P4.50-LS6.5
- U2: value TPS54331DR -> ~; footprint PCM_JLCPCB:SOIC-8_L5.0-W4.0-P1.27-LS6.0-BL -> RP2350_Console_Parts_lib:VSON-14_L4.0-W3.0-P0.50-BL-EP_TI_DSJ
- U3: moved to B.Cu
- moved C32 19.7 mm to (103.5, 156.5)
- moved C14 18.2 mm to (95.5, 121.4), turned to -45 degrees
- moved C4 16.9 mm to (71.5, 121.0)
- moved C5 16.7 mm to (114.2, 115.6), turned to 0 degrees
- moved C35 16.6 mm to (68.7, 121.9)
- moved C31 14.9 mm to (83.5, 155.4)
- moved C3 13.9 mm to (94.4, 129.2), turned to 90 degrees
- moved R15 13.8 mm to (98.8, 119.6), turned to 180 degrees
- moved C30 13.2 mm to (91.5, 126.8), turned to 135 degrees
- moved R16 13.2 mm to (98.8, 120.5), turned to 180 degrees
- moved R11 12.1 mm to (79.2, 129.1), turned to 45 degrees
- moved R2 12.1 mm to (137.0, 128.5)
- moved U3 11.9 mm to (82.9, 123.4), turned to -135 degrees
- moved R10 11.3 mm to (80.7, 129.8), turned to 90 degrees
- moved C1 10.2 mm to (114.2, 116.9), turned to 0 degrees
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Connections:
- C1 pad 1: +3V3 -> VSYS
- C5 pad 1: Net-(U2-SS) -> VSYS
- L2 pad 1: Net-(U2-PH) -> Net-(L2-Pad1)
- L2 pad 2: +3V3 -> Net-(L2-Pad2)
- R14 pad 1: Net-(U2-COMP) -> Net-(U2-FB)
- R14 pad 2: Net-(C24-Pad1) -> GND
- R15 pad 1: +3V3 -> Net-(U4-ISET)
- R15 pad 2: Net-(U2-VSENSE) -> GND
- R16 pad 1: Net-(U2-VSENSE) -> Net-(U4-PRE-TERM)
- U2 pad 2: VBUS -> GND
- U2 pad 3: unconnected-(U2-EN-Pad3) -> Net-(U2-FB)
- U2 pad 4: Net-(U2-SS) -> +3V3
- U2 pad 5: Net-(U2-VSENSE) -> +3V3
- U2 pad 6: Net-(U2-COMP) -> Net-(L2-Pad1)
- U2 pad 7: GND -> Net-(L2-Pad1)
- U2 pad 8: Net-(U2-PH) -> Net-(L2-Pad2)
Routing:
- net +3V3: track 107.1 -> 14.9 mm, vias 1 -> 0
- net /RUN: track 39.5 -> 0.00 mm, vias 2 -> 0
- net GND: track 46.0 -> 12.0 mm, vias 38 -> 26
- net /USER_LED: track 31.6 -> 0.00 mm, vias 2 -> 0
- net /LQ_BUT: track 31.5 -> 0.00 mm
- net /~{USB_BOOT}: track 30.9 -> 0.00 mm
- net /RQ_BUT: track 29.6 -> 0.00 mm
- net +1V1: track 36.4 -> 8.21 mm, vias 10 -> 4
- net VSYS: track 0.00 -> 19.3 mm
- net VBUS: track 0.00 -> 18.6 mm
- net /QSPI2_SS: track 18.6 -> 0.00 mm
- net /RQ_P2: track 18.2 -> 0.00 mm
- net /LQ_P1: track 16.7 -> 0.00 mm
- net /RQ_P1: track 15.7 -> 0.00 mm
- net /LQ_P2: track 14.8 -> 0.00 mm
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- added copper zone on F.Cu, net Net-(L2-Pad1)
- added copper zone on F.Cu, net Net-(L2-Pad2)
- added copper zone on F.Cu, net VSYS
- removed copper zone on F.Cu, net VBUS

Commit message: updates to pcb
Parts:
- moved C13 32.8 mm to (138.9, 135.9)
- moved C34 32.8 mm to (138.9, 136.8)
- moved R21 32.8 mm to (136.7, 140.0)
- moved R22 32.8 mm to (139.8, 141.3)
- moved R6 32.8 mm to (134.3, 136.1)
- moved C19 32.8 mm to (137.2, 141.7)
- moved C33 32.8 mm to (137.0, 134.8)
- moved C6 32.8 mm to (133.0, 137.8)
- moved X1 24.2 mm to (105.3, 137.9), turned to 45 degrees
- moved C22 21.1 mm to (104.4, 135.3), turned to 45 degrees
- moved C14 21.0 mm to (113.6, 132.0)
- moved C29 20.4 mm to (102.8, 136.9), turned to -135 degrees
- moved C8 18.4 mm to (103.0, 133.8), turned to -45 degrees
- moved R13 18.0 mm to (102.3, 134.5), turned to 135 degrees
- moved C12 17.7 mm to (101.4, 135.5), turned to -45 degrees
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Routing:
- net /USB_D+: track 14.6 -> 2.97 mm
- net /USB_D-: track 14.3 -> 2.94 mm
- net Net-(U1-USB_DM): track 5.18 -> 2.85 mm
- net /QSPI_SD2: vias 1 -> 2
- net GND: vias 26 -> 25

Commit message: v2.0 design files
Parts:
- removed D2: Green, PCM_JLCPCB:D_0805
- removed J5: Conn_01x08_MountingPin, RP2350_Console_Parts_lib:Seeed 1.69 Inch LCD Module
- removed R8: 100Ω, PCM_JLCPCB:R_0402
- added C20: 100nF, PCM_JLCPCB:C_0402, F.Cu at (83.4, 130.4)
- added C21: 100nF, PCM_JLCPCB:C_0402, F.Cu at (83.4, 126.4)
- added CN1: S2B-PH-SM4-TB(LF)(SN), easyeda2kicad:CONN-SMD_P2.00_S2B-PH-SM4-TB-LF-SN, F.Cu at (124.4, 120.9)
- added D1: Yellow, easyeda2kicad:LED0603-R-RD_AMBER, F.Cu at (103.1, 122.5)
- added J1: Conn_01x08_MountingPin, RP2350_Console_Parts_lib:Seeed 1.69 Inch LCD Module, F.Cu at (90.0, 146.6)
- added LED1: TC5050RGBF08-3CJH-AF53A, easyeda2kicad:LED-SMD_6P-L5.0-W5.0-TL_TC5050RGBF08, F.Cu at (58.7, 117.7)
- added R23: 55R, PCM_JLCPCB:R_0603, F.Cu at (56.1, 122.9)
- added R24: 1kΩ, PCM_JLCPCB:R_0402, F.Cu at (105.5, 124.4)
- added R25: 1kΩ, PCM_JLCPCB:R_0402, F.Cu at (105.9, 122.1)
- added R26: 15Ω, PCM_JLCPCB:R_0603, F.Cu at (57.4, 123.0)
- added TP1: TestPoint, TestPoint:TestPoint_Pad_1.0x1.0mm, F.Cu at (118.6, 113.5)
- added TP2: TestPoint, TestPoint:TestPoint_Pad_1.0x1.0mm, F.Cu at (97.0, 115.3)
- added TP3: TestPoint, TestPoint:TestPoint_Pad_1.0x1.0mm, F.Cu at (101.7, 133.0)
- added TP4: TestPoint, TestPoint:TestPoint_Pad_1.0x1.0mm, F.Cu at (80.9, 142.8)
- D5: value Red -> Blue; footprint PCM_JLCPCB:D_0603 -> easyeda2kicad:LED0603-FD_BLUE
- R15: value 1kΩ -> 560Ω; footprint PCM_JLCPCB:R_0402 -> PCM_JLCPCB:R_0603
- R19: value 47kΩ -> 10kΩ; footprint PCM_JLCPCB:R_0603 -> PCM_JLCPCB:R_0402
- R20: value 1.5kΩ -> 15Ω
- R3, R7: value 27Ω -> 27R; footprint PCM_JLCPCB:R_0603 -> easyeda2kicad:R0201
- moved R20 53.5 mm to (54.8, 123.0)
- moved R22 43.2 mm to (99.7, 125.1)
- moved C13 43.0 mm to (96.6, 128.4)
- moved C34 42.6 mm to (96.6, 132.4)
- moved R6 41.7 mm to (95.7, 120.3)
- moved C19 41.5 mm to (99.7, 124.0)
- moved C33 40.7 mm to (96.6, 129.3)
- moved C6 40.4 mm to (95.7, 122.2)
- moved R21 39.4 mm to (99.7, 126.4), turned to 180 degrees
- moved C35 31.5 mm to (98.3, 132.6), turned to 90 degrees
- moved C14 30.4 mm to (83.4, 128.6), turned to 180 degrees
- moved C32 24.6 mm to (83.3, 142.5), turned to 90 degrees
- moved C30 22.9 mm to (67.4, 124.0), turned to 90 degrees
- moved C4 21.1 mm to (86.9, 135.4), turned to -135 degrees
- moved U5 20.6 mm to (71.7, 122.2), turned to 0 degrees
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Connections:
- C1 pad 1: VSYS -> +BATT
- C5 pad 1: VSYS -> +BATT
- R19 pad 2: VSYS -> GND
- R20 pad 1: Net-(D5-Pad2) -> /RGB_LED_G
- R20 pad 2: VSYS -> Net-(LED1-+-Pad1)
- R21 pad 1: VIN -> +BATT
- R3 pad 1: Net-(U1-USB_DM) -> Net-(U1-USB_DP)
- R3 pad 2: /USB_D- -> /USB_D+
- R7 pad 1: Net-(U1-USB_DP) -> Net-(U1-USB_DM)
- R7 pad 2: /USB_D+ -> /USB_D-
- SW6 pad 1: VSYS -> +BATT
- U1 pad 13: /GPIO14 -> /RGB_LED_B
- U1 pad 16: /GPIO16 -> /RGB_LED_R
- U1 pad 17: /GPIO17 -> /RGB_LED_G
- U1 pad 18: /GPIO18 -> /RQ_BUT
- U1 pad 19: /GPIO19 -> /RQ_P1
- U1 pad 20: /GPIO20 -> /RQ_P2
- U1 pad 21: /RQ_BUT -> /Screen_CS
- U1 pad 22: /RQ_P1 -> /Screen_CLK
- U1 pad 23: /RQ_P2 -> /Screen_DIN
- U1 pad 25: /Screen_BL -> /Screen_DC
- U1 pad 26: /Screen_RST -> unconnected-(U1-GPIO25-Pad26)
- U1 pad 27: /Screen_DC -> unconnected-(U1-GPIO26-Pad27)
- U1 pad 36: /GPIO28 -> /Screen_RST
- U1 pad 37: /Screen_CS -> /Screen_BL
- U1 pad 38: /Screen_CLK -> /LQ_P1
- U1 pad 39: /Screen_DIN -> /LQ_P2
- U1 pad 40: /GPIO32 -> /LQ_BUT
- U1 pad 42: /LQ_P1 -> unconnected-(U1-GPIO33-Pad42)
- U1 pad 43: /LQ_P2 -> unconnected-(U1-GPIO34-Pad43)
- U1 pad 44: /LQ_BUT -> unconnected-(U1-GPIO35-Pad44)
- U2 pad 10: VSYS -> +BATT
- U2 pad 11: VSYS -> +BATT
- U4 pad 10: VSYS -> +BATT
- U4 pad 8: unconnected-(U4-CHG#-Pad8) -> Net-(U4-CHG#)
Routing:
- net +3V3: track 14.9 -> 240.9 mm, vias 0 -> 1
- net /USER_LED: track 0.00 -> 45.5 mm
- net /RUN: track 0.00 -> 38.1 mm
- net /RGB_LED_G: track 0.00 -> 36.4 mm
- net /RGB_LED_R: track 0.00 -> 35.2 mm
- net /RGB_LED_B: track 0.00 -> 35.0 mm
- net /QSPI2_SS: track 0.00 -> 33.8 mm
- net /LQ_BUT: track 0.00 -> 33.2 mm
- net /RQ_BUT: track 0.00 -> 30.5 mm
- net +BATT: track 0.00 -> 30.0 mm
- net /LQ_P1: track 0.00 -> 19.6 mm
- net VSYS: track 19.3 -> 0.00 mm
- net /RQ_P2: track 0.00 -> 17.8 mm
- net /LQ_P2: track 0.00 -> 17.1 mm
- net /RQ_P1: track 0.00 -> 15.9 mm
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- added copper zone on F.Cu, net +BATT
- removed copper zone on F.Cu, net VSYS
