File: Hardware/RP2350b_Console/RP2350b_Console.kicad_sch (KiCad schematic)
At the start: 63 parts, among them J2 Connector, USB-TYPE-C-16P, J5 Conn_01x08_MountingPin, SW1 SW_Push, SW2 SW_Push, SW3 RotaryEncoder_Switch_MP, SW4 RotaryEncoder_Switch_MP, U1 RP2350_80QFN, U2 TPS54331DR, U3 LY68L6400SLIT, U5 W25Q128, X1 ABM8-272-T3

Commit message: updates
Parts:
- removed C1, C27: 100uF, PCM_JLCPCB:C_1206, symbol PCM_JLCPCB-Capacitors:1206,100uF
- removed C23: 100nF, PCM_JLCPCB:C_0402, symbol PCM_JLCPCB-Capacitors:0402,100nF,(2)
- removed C24: 1nF, PCM_JLCPCB:C_0402, symbol PCM_JLCPCB-Capacitors:0402,1nF
- removed C25: 10pF, PCM_JLCPCB:C_0402, symbol PCM_JLCPCB-Capacitors:0402,10pF
- removed C26: 22uF, PCM_JLCPCB:C_0805, symbol PCM_JLCPCB-Capacitors:0805,22uF
- removed C5: 2.7nF, PCM_JLCPCB:C_0603, symbol PCM_JLCPCB-Capacitors:0603,2.7nF
- removed D1: SS24F, PCM_JLCPCB:D_SMAF, symbol PCM_JLCPCB-Diodes:Schottky,SS24F
- removed L2: 2.7uH, Inductor_SMD:IND-SMD_L5.0-W5.0_FNR50XXS, symbol Custom:SWPA5040S2R7NT
- removed R14: 24kΩ, PCM_JLCPCB:R_0402, symbol PCM_JLCPCB-Resistors:0402,24kΩ
- removed R15: 10kΩ, PCM_JLCPCB:R_0402, symbol PCM_JLCPCB-Resistors:0402,10kΩ
- removed R16: 3.3kΩ, PCM_JLCPCB:R_0402, symbol PCM_JLCPCB-Resistors:0402,3.3kΩ
- removed U2: TPS54331DR, PCM_JLCPCB:SOIC-8_L5.0-W4.0-P1.27-LS6.0-BL, symbol PCM_JLCPCB-Power:DC-DC, Buck, 3.5-28VIN, 3A, 0.8+VOUT
- added C1, C10, C16, C17: 22uF, PCM_JLCPCB:C_0603, symbol PCM_JLCPCB-Capacitors:0603,22uF
- added C18: 1uF, PCM_JLCPCB:C_0402, symbol PCM_JLCPCB-Capacitors:0402,1uF
- added C19, C7: 100nF, PCM_JLCPCB:C_0402, symbol PCM_JLCPCB-Capacitors:0402,100nF,(2)
- added C5, C9: 10uF, PCM_JLCPCB:C_0603, symbol PCM_JLCPCB-Capacitors:0603,10uF
- added D5: Red, PCM_JLCPCB:D_0603, symbol PCM_JLCPCB-Diodes:LED,0603,Red
- added L2: 1.5uH, RP2350_Console_Parts_lib:IND-SMD_L4.0-W4.0-A, symbol RP2350_Console_Parts_lib:XFL4020-152MEC
- added R14, R9: 1MΩ, PCM_JLCPCB:R_0603, symbol PCM_JLCPCB-Resistors:0603,1MΩ
- added R15: 1kΩ, PCM_JLCPCB:R_0402, symbol PCM_JLCPCB-Resistors:0402,1kΩ
- added R16: 2kΩ, PCM_JLCPCB:R_0402, symbol PCM_JLCPCB-Resistors:0402,2kΩ
- added R19: 47kΩ, PCM_JLCPCB:R_0603, symbol PCM_JLCPCB-Resistors:0603,47kΩ
- added R20: 1.5kΩ, PCM_JLCPCB:R_0603, symbol PCM_JLCPCB-Resistors:0603,1.5kΩ
- added R21, R22: 100kΩ, PCM_JLCPCB:R_0603, symbol PCM_JLCPCB-Resistors:0603,100kΩ
- added SW6: ~, RP2350_Console_Parts_lib:SW-TH_MK-12D18-G040, symbol RP2350_Console_Parts_lib:MK-12D18-G040
- added U2: ~, RP2350_Console_Parts_lib:VSON-14_L4.0-W3.0-P0.50-BL-EP_TI_DSJ, symbol RP2350_Console_Parts_lib:TPS63020DSJR
- added U4: ~, RP2350_Console_Parts_lib:MSOP-10_L3.0-W3.0-P0.50-LS5.0-BL-EP, symbol RP2350_Console_Parts_lib:BQ24092DGQR
- J5: footprint Display:Seeed 1.69 Inch LCD Module -> RP2350_Console_Parts_lib:Seeed 1.69 Inch LCD Module
- L1: footprint Inductor_SMD:IND-SMD_L2.0-W1.6_AOTA-B201610S3R3-101-T -> RP2350_Console_Parts_lib:IND-SMD_L2.0-W1.6_AOTA-B201610S3R3-101-T
- SW1, SW2: footprint Button_Switch_THT:SW_1825910-6-4 -> RP2350_Console_Parts_lib:SW-TH_4P-L6.0-W6.0-P4.50-LS6.5
Connections:
- net +3V3: now also C10.1, C16.1, C9.1, R9.1, U2.4 (VOUT), U2.5 (VOUT)
- net GND: now also C1.2, C10.2, C16.2, C17.2, C18.2, C19.2, C5.2, C7.2, C9.2, R14.2, R15.2, R16.2, R22.2, SW6.3, U2.13 (PS/SYNC), U2.15 (PGND), U2.2 (GND), U4.11 (EP), U4.3 (VSS), U4.7 (ISET2)
- net VBUS: now also C17.1, C18.1, U4.1 (IN)
- new net: R19.1, U4.9 (TS)
- new net: D5.1, U4.5 (PG#)
- new net: D5.2, R20.1
- new net: R14.1, R9.2, U2.3 (FB)
- new net: SW6.2, U2.12 (EN)
- new net: L2.1, U2.6 (L2), U2.7 (L2)
- new net: L2.2, U2.8 (L1), U2.9 (L1)
- new net: C7.1, U2.1 (VINA)
- new net: R15.1, U4.2 (ISET)
- new net: R16.1, U4.4 (PRE-TERM)
- new net Sense: C19.1, R21.2, R22.1
- new net VIN: R21.1
- new net VSYS: C1.1, C5.1, R19.2, R20.2, SW6.1, U2.10 (VIN), U2.11 (VIN), U4.10 (OUT)
- no-connect marks 3 -> 5
Other:
- moved on the sheet: J2, R12, R5

Commit message: v2.0 design files
Parts:
- removed D2: Green, PCM_JLCPCB:D_0805, symbol PCM_JLCPCB-Diodes:LED,0805,Green
- removed J5: Conn_01x08_MountingPin, RP2350_Console_Parts_lib:Seeed 1.69 Inch LCD Module, symbol Connector_Generic_MountingPin:Conn_01x08_MountingPin
- removed R15: 1kΩ, PCM_JLCPCB:R_0402, symbol PCM_JLCPCB-Resistors:0402,1kΩ
- removed R19: 47kΩ, PCM_JLCPCB:R_0603, symbol PCM_JLCPCB-Resistors:0603,47kΩ
- removed R20: 1.5kΩ, PCM_JLCPCB:R_0603, symbol PCM_JLCPCB-Resistors:0603,1.5kΩ
- removed R3, R7: 27Ω, PCM_JLCPCB:R_0603, symbol PCM_JLCPCB-Resistors:0603,27Ω
- removed R8: 100Ω, PCM_JLCPCB:R_0402, symbol PCM_JLCPCB-Resistors:0402,100Ω
- added C20, C21: 100nF, PCM_JLCPCB:C_0402, symbol PCM_JLCPCB-Capacitors:0402,100nF,(2)
- added CN1: S2B-PH-SM4-TB(LF)(SN), easyeda2kicad:CONN-SMD_P2.00_S2B-PH-SM4-TB-LF-SN, symbol easyeda2kicad:S2B-PH-SM4-TB(LF)(SN)
- added D1: Yellow, easyeda2kicad:LED0603-R-RD_AMBER, symbol PCM_JLCPCB-Diodes:LED,0603,Red
- added J1: Conn_01x08_MountingPin, RP2350_Console_Parts_lib:Seeed 1.69 Inch LCD Module, symbol Connector_Generic_MountingPin:Conn_01x08_MountingPin
- added LED1: TC5050RGBF08-3CJH-AF53A, easyeda2kicad:LED-SMD_6P-L5.0-W5.0-TL_TC5050RGBF08, symbol easyeda2kicad:TC5050RGBF08-3CJH-AF53A
- added R15: 560Ω, PCM_JLCPCB:R_0603, symbol PCM_JLCPCB-Resistors:0603,560Ω
- added R19: 10kΩ, PCM_JLCPCB:R_0402, symbol PCM_JLCPCB-Resistors:0402,10kΩ
- added R20, R26: 15Ω, PCM_JLCPCB:R_0603, symbol PCM_JLCPCB-Resistors:0603,15Ω
- added R23: 55R, PCM_JLCPCB:R_0603, symbol Device:R
- added R24, R25: 1kΩ, PCM_JLCPCB:R_0402, symbol PCM_JLCPCB-Resistors:0402,1kΩ
- added R3, R7: 27R, easyeda2kicad:R0201, symbol Device:R
- added TP1, TP2, TP3, TP4: TestPoint, TestPoint:TestPoint_Pad_1.0x1.0mm, symbol Connector:TestPoint
- D5: value Red -> Blue; footprint PCM_JLCPCB:D_0603 -> easyeda2kicad:LED0603-FD_BLUE
Connections:
- net GPIO18 is gone; now on net RQ_BUT: U1.18 (GPIO18)
- net GPIO19 is gone; now on net RQ_P1: U1.19 (GPIO19)
- net GPIO20 is gone; now on net RQ_P2: U1.20 (GPIO20)
- net GPIO28 is gone; now on net Screen_RST: U1.36 (GPIO28)
- net GPIO32 is gone; now on net LQ_BUT: U1.40 (GPIO32)
- net VSYS is gone; now on net +BATT: C1.1, C5.1, SW6.1, U2.10 (VIN), U2.11 (VIN), U4.10 (OUT)
- net +3V3: now also C20.1, C21.1, J1.8 (Pin_8), TP3.1, TP4.1
- net GND: now also C20.2, C21.2, CN1.1, CN1.3, CN1.4, J1.7 (Pin_7), J1.MP (MountPin), LED1.4 (-), LED1.5 (-), LED1.6 (-), R15.2, R19.2
- net LQ_BUT: no longer U1.44 (GPIO35)
- net LQ_P1: now also U1.38 (GPIO30); no longer U1.42 (GPIO33)
- net LQ_P2: now also U1.39 (GPIO31); no longer U1.43 (GPIO34)
- net RQ_BUT: no longer U1.21 (GPIO21)
- net RQ_P1: no longer U1.22 (GPIO22)
- net RQ_P2: no longer U1.23 (GPIO23)
- net Screen_BL: now also U1.37 (GPIO29), J1.1 (Pin_1); no longer U1.25 (GPIO24)
- net Screen_CLK: now also U1.22 (GPIO22), J1.5 (Pin_5); no longer U1.38 (GPIO30)
- net Screen_CS: now also U1.21 (GPIO21), J1.6 (Pin_6); no longer U1.37 (GPIO29)
- net Screen_DC: now also U1.25 (GPIO24), J1.3 (Pin_3); no longer U1.27 (GPIO26)
- net Screen_DIN: now also U1.23 (GPIO23), J1.4 (Pin_4); no longer U1.39 (GPIO31)
- net Screen_RST: now also J1.2 (Pin_2); no longer U1.26 (GPIO25)
- net USB_D+: now also R3.2
- net USB_D-: now also R7.2
- net VBUS: now also TP2.1
- net at U4.9 (TS): now also R19.1
- net at D5.2: now also R24.1
- net at U1.67 (USB_DP): now also R3.1
- net at U1.66 (USB_DM): now also R7.1
- net at U4.2 (ISET): now also R15.1
- net at U4.8 (CHG#): now also D1.1
- net GPIO14 renamed RGB_LED_B
- net RGB_LED_B: now also R26.1
- net GPIO16 renamed RGB_LED_R
- net RGB_LED_R: now also R23.1
- net GPIO17 renamed RGB_LED_G
- net RGB_LED_G: now also R20.1
- net VIN renamed +BATT
- net +BATT: now also CN1.2, R24.2, R25.2, TP1.1
- new net: LED1.1 (+), R20.2
- new net: LED1.3 (+), R26.2
- new net: D1.2, R25.1
- new net: LED1.2 (+), R23.2
- no-connect marks 5 -> 4
