File: HardwareV2/crystal.kicad_sch (KiCad schematic)
At the start: 4 parts, among them U6 ABM8-272-T3

Commit message: initial v2 pcb layout minus passives
Parts:
- C4, C5: footprint (none) -> Capacitor_SMD:C_0805_2012Metric
- R8: footprint (none) -> Resistor_SMD:R_0805_2012Metric
- U6: footprint parts_lib:CRYSTAL-SMD_4P-L3.2-W2.5-BL-2 -> RP2350b_parts_layout:CRYSTAL-SMD_4P-L3.2-W2.5-BL-2
Changed lines of the file:
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@@
 			)
 		)
-		(property "Footprint" ""
+		(property "Footprint" "Capacitor_SMD:C_0805_2012Metric"
 			(at 163.83 91.44 0)
 			(effects
@@
 			)
 		)
-		(property "Footprint" ""
+		(property "Footprint" "Resistor_SMD:R_0805_2012Metric"
 			(at 148.59 96.52 0)
 			(effects
@@
 			)
 		)
-		(property "Footprint" "parts_lib:CRYSTAL-SMD_4P-L3.2-W2.5-BL-2"
+		(property "Footprint" "RP2350b_parts_layout:CRYSTAL-SMD_4P-L3.2-W2.5-BL-2"
 			(at 133.35 100.33 0)
 			(effects
@@
 			)
 		)
-		(property "Footprint" ""
+		(property "Footprint" "Capacitor_SMD:C_0805_2012Metric"
 			(at 143.51 100.33 0)
 			(effects
