File: HardwareV2/memory.kicad_sch (KiCad schematic)
At the start: 2 parts, among them U4 W25Q128JVSIQTR, U5 LY68L6400SLIT

Commit message: initial v2 pcb layout minus passives
Parts:
- U4: footprint parts_lib:SOIC-8_L5.3-W5.3-P1.27-LS8.0-BL -> RP2350b_parts_layout:SOIC-8_L5.3-W5.3-P1.27-LS8.0-BL
- U5: footprint parts_lib:SOP-8_L4.9-W3.9-P1.27-LS6.0-BL -> RP2350b_parts_layout:SOP-8_L4.9-W3.9-P1.27-LS6.0-BL
Changed lines of the file:
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@@
 			)
 		)
-		(property "Footprint" "parts_lib:SOP-8_L4.9-W3.9-P1.27-LS6.0-BL"
+		(property "Footprint" "RP2350b_parts_layout:SOP-8_L4.9-W3.9-P1.27-LS6.0-BL"
 			(at 80.772 132.08 0)
 			(effects
@@
 			)
 		)
-		(property "Footprint" "parts_lib:SOIC-8_L5.3-W5.3-P1.27-LS8.0-BL"
+		(property "Footprint" "RP2350b_parts_layout:SOIC-8_L5.3-W5.3-P1.27-LS8.0-BL"
 			(at 73.66 74.93 0)
 			(effects
